File: PC104_io_conn.kicad_sch (KiCad schematic)
At the start: 2 parts, among them J1 ESQ-126-39-G-D, J2 ESQ-126-39-G-D

Commit message: Change the connector, power cleanups
Change the PC104 connector. The CSKB specifies ESQ-126-39-G-D, which
have 12.19mm pins.  This leaves around 3mm of pin exposed between the
boards.  This design has ESQ-126-38-G-D PC104 which will leave no space.

Rework the power to a fairly common setup.

Signed-off-by: Corey Minyard <corey@minyard.net>
Parts:
- added R10, R12, R13, R14, R15, R3, R4, R8: 0Ω, Resistor_SMD:R_0603_1608Metric_Pad0.98x0.95mm_HandSolder, symbol Device:R
- J1, J2: value ESQ-126-39-G-D -> ESQ-126-38-G-D
Connections:
- net 3.3V_p: now also R4.2
- net 5V_p: now also R8.1
- net 3.3V_S1_p renamed 3V3_S1
- net 3V3_S1: now also R13.1
- net 3.3V_S2_p renamed 3V3_S2
- net 3V3_S2: now also R14.1
- net 3.3V_S3_p renamed 3V3_S3
- net 3V3_S3: now also R15.1
- net 5V_S1_p renamed 5V_S1
- net 5V_S1: now also R12.2
- net 5V_S2_p renamed 5V_S2
- net 5V_S2: now also R10.2
- net 5V_S3_p renamed 5V_S3
- net 5V_S3: now also R3.2
- new net 3.3V_IN: R13.2, R14.2, R15.2, R4.1
- new net 5V_IN: R10.1, R12.1, R3.1, R8.2
