File: PacSatBaseBoard.kicad_pcb (KiCad board)
At the start: 6 copper layers, 90.2 x 95.9 mm, 33 parts, among them J1 ESQ-126-39-G-D, J2 ESQ-126-39-G-D, J3 FTSH-105-01-L-DV-K, J4 TS-103-G-A, J5 HTSW-102-07-G-S, J7 G125-MH11005L1P, J8 Conn_01x02_Pin

Commit message: Change the connector, power cleanups
Change the PC104 connector. The CSKB specifies ESQ-126-39-G-D, which
have 12.19mm pins.  This leaves around 3mm of pin exposed between the
boards.  This design has ESQ-126-38-G-D PC104 which will leave no space.

Rework the power to a fairly common setup.

Signed-off-by: Corey Minyard <corey@minyard.net>
Parts:
- added R10: 0Ω, Resistor_SMD:R_0603_1608Metric_Pad0.98x0.95mm_HandSolder, F.Cu at (76.4, -79.0)
- added R12: 0Ω, Resistor_SMD:R_0603_1608Metric_Pad0.98x0.95mm_HandSolder, F.Cu at (73.8, -78.9)
- added R13: 0Ω, Resistor_SMD:R_0603_1608Metric_Pad0.98x0.95mm_HandSolder, B.Cu at (73.8, -78.9)
- added R14: 0Ω, Resistor_SMD:R_0603_1608Metric_Pad0.98x0.95mm_HandSolder, B.Cu at (76.4, -79.0)
- added R15: 0Ω, Resistor_SMD:R_0603_1608Metric_Pad0.98x0.95mm_HandSolder, B.Cu at (79.0, -78.9)
- added R3: 0Ω, Resistor_SMD:R_0603_1608Metric_Pad0.98x0.95mm_HandSolder, F.Cu at (79.0, -78.9)
- added R4: 0Ω, Resistor_SMD:R_0603_1608Metric_Pad0.98x0.95mm_HandSolder, F.Cu at (51.4, -80.6)
- added R8: 0Ω, Resistor_SMD:R_0603_1608Metric_Pad0.98x0.95mm_HandSolder, F.Cu at (47.0, -78.9)
- J1, J2: value ESQ-126-39-G-D -> ESQ-126-38-G-D; footprint PacSatDev_misc:CONN_ESQ-126-39-G-D_SAI -> Local_Footprints:CONN_ESQ-126-39-G-D_SAI
- J3: footprint PacSatDev_samtec:FTSH-105-01-L-DV-K -> Local_Footprints:FTSH-105-01-L-DV-K
- J4: value TS-103-G-A -> TSW-103-08-F-S-RA; footprint Local_Footprints:CON3_1X3_TU_HTS_SAI -> Local_Footprints:CON3_1X3_TR_TSW_SAI
- J5: footprint PacSatDev_misc:CON2_1X2_TU_TSW -> Local_Footprints:CON2_1X2_TU_TSW
- J7: footprint PacSatDev_misc:G125-MH11005L1P -> Local_Footprints:G125-MH11005L1P
- moved J5 47.0 mm to (82.4, -83.8), turned to 90 degrees
- moved J3 41.2 mm to (4.05, -62.8), turned to 90 degrees
- moved R6 36.0 mm to (14.5, -62.1)
- moved C136 36.0 mm to (14.4, -58.1)
- moved R5 36.0 mm to (14.5, -64.1)
- moved R7 36.0 mm to (14.5, -60.1)
- moved D2 32.3 mm to (65.6, -75.8)
- moved C114 31.5 mm to (73.7, -75.8)
- moved L2 26.7 mm to (69.6, -77.4), turned to 90 degrees
- moved R2 17.0 mm to (62.9, -76.8), turned to 90 degrees
- moved J4 7.56 mm to (10.7, -79.5)
Connections:
- net /Antenna Control/I2CA_SCL renamed I2CA_SCL
- net /Antenna Control/I2CA_SDA renamed I2CA_SDA
- net /Antenna Control/I2CB_SCL renamed I2CB_SCL
- net /Antenna Control/I2CB_SDA renamed I2CB_SDA
- net 3.3V_p renamed /PC104_IO/3.3V_p
- net 5V_p renamed /PC104_IO/5V_p
- J1 pad 47: 5V_S1_p -> /PC104_IO/5V_S1
- J1 pad 48: 3.3V_S1_p -> /PC104_IO/3V3_S1
- J1 pad 49: 5V_S2_p -> /PC104_IO/5V_S2
- J1 pad 50: 3.3V_S2_p -> /PC104_IO/3V3_S2
- J1 pad 51: 5V_S3_p -> /PC104_IO/5V_S3
- J1 pad 52: 3.3V_S3_p -> /PC104_IO/3V3_S3
Routing:
- net 5V_IN: track 0.00 -> 37.4 mm
- net 3.3V_IN: track 0.00 -> 29.6 mm, vias 0 -> 4
- net /PC104_IO/5V_p: track 0.00 -> 27.1 mm, vias 0 -> 2
- net /PC104_IO/3.3V_p: track 0.00 -> 23.5 mm, vias 0 -> 2
- net /PC104_IO/3V3_S3: track 0.00 -> 6.50 mm
- net /PC104_IO/3V3_S1: track 0.00 -> 6.49 mm
- net /PC104_IO/3V3_S2: track 0.00 -> 6.46 mm
- net +5V: track 0.00 -> 5.81 mm
- net /PC104_IO/5V_S3: track 0.00 -> 3.96 mm
- net /PC104_IO/5V_S1: track 0.00 -> 3.93 mm
- net /PC104_IO/5V_S2: track 0.00 -> 3.90 mm
- net GND: track 0.00 -> 2.82 mm, vias 0 -> 3
- net Net-(D2-K): track 0.00 -> 1.81 mm
